Commit message: Add files via upload
Actualizacion

File: arips_ros/arips_arm_description/urdf/arips_arm.xacro (robot description, xacro)
@@ -28,4 +28,13 @@
   <xacro:property name="link6_radius" value="0.01" />
   <xacro:property name="gripper_open_angle" value="0.06" />
+  <link name="world">
+    <origin xyz="0.0 0.0 0.0" rpy="0 0 0"/>
+  </link>
+  <joint name="base_joint" type="fixed">
+    <parent link="world"/>
+    <child link="arm_base_link"/>
+    <!--origin xyz="0.0 0.0 0.0" rpy="0 0 -1.5707"/--> <!--  - - - - - - OJO MUCHO OJO - - - -  - - - -->
+    <origin xyz="0.0 0.0 0.0" rpy="0 0 0"/> <!--  - - - - - - OJO MUCHO OJO - - - -  - - - -->
+  </joint>
   <link name="arm_base_link">
     <visual>

File: arips_ros/arips_arm_description/urdf/definir_hardware_ros2_control.xacro (robot description, xacro)
@@ -3,5 +3,5 @@
   <xacro:arg name="dedo_mimic" default="false" />
   <!--xacro:arg name="use_sim_time" default="true" /-->
-  <xacro:macro name="definir_hardware" params="name use_sim_time:=^|true">
+  <xacro:macro name="definir_hardware" params="name use_sim_time">
     <ros2_control name="${name}" type="system">
      <hardware>
@@ -24,11 +24,12 @@
           <param name="multiplier">1</param>
         </xacro:if>
+        <xacro:unless value="$(arg dedo_mimic)">
         <command_interface name="position">
-          <param name="min">-1</param>
-          <param name="max">1</param>
+          <param name="min">10</param>
+          <param name="max">1000</param>
         </command_interface>
         <command_interface name="velocity">
-          <param name="min">-10</param>
-          <param name="max">10</param>
+          <param name="min">0</param>
+          <param name="max">100</param>
         </command_interface>
         <!--command_interface name="acceleration">
@@ -39,4 +40,5 @@
         <state_interface name="velocity"/>
         <!--state_interface name="acceleration"/-->
+        </xacro:unless>
       </joint>
     </xacro:macro>

Commit message: Add files via upload
Actualizacion

File: arips_ros/arips_arm_description/urdf/arips_arm.xacro (robot description, xacro)
@@ -119,5 +119,5 @@
     <axis xyz="0 0 1"/>
     <origin xyz="0 0 ${link1_height}"/>
-    <limit effort="1000.0" lower="${-pi*0.45}" upper="${pi*0.45}" velocity="1.0"/>
+    <limit effort="1000.0" lower="-2.09" upper="2.09" velocity="500"/> <!-- 2.09 = 120 grados -->
   </joint>
   <joint name="joint2" type="revolute">
@@ -126,5 +126,5 @@
     <axis xyz="0 1 0"/>
     <origin xyz="0.02 0 ${link2_height}"/>
-    <limit effort="1000.0" lower="-0.95" upper="2.1" velocity="1.0"/>
+    <limit effort="1000.0" lower="-2.09" upper="2.09" velocity="500"/>
   </joint>
   <joint name="joint3" type="revolute">

File: arips_ros/arips_arm_description/urdf/definir_hardware_ros2_control.xacro (robot description, xacro)
@@ -24,12 +24,11 @@
           <param name="multiplier">1</param>
         </xacro:if>
-        <xacro:unless value="$(arg dedo_mimic)">
         <command_interface name="position">
-          <param name="min">10</param>
-          <param name="max">1000</param>
+          <param name="min">-2.09</param>
+          <param name="max">2.09</param>
         </command_interface>
         <command_interface name="velocity">
           <param name="min">0</param>
-          <param name="max">100</param>
+          <param name="max">5000</param>
         </command_interface>
         <!--command_interface name="acceleration">
@@ -40,5 +39,4 @@
         <state_interface name="velocity"/>
         <!--state_interface name="acceleration"/-->
-        </xacro:unless>
       </joint>
     </xacro:macro>
