Commit message: Add files via upload
4 abril 2024

File: arips_ros/arips_arm_description/urdf/arips_arm.urdf (robot description, URDF)
Before this commit: robot arips_arm, 10 links, 9 joints
Joints:
- joint joint1: limit lower=-1.40 upper=1.40 effort=1000.0 velocity=1.0 -> lower=-1.40 upper=1.40 effort=100.0 velocity=1.0
- joint joint2: limit lower=-0.95 upper=2.1 effort=1000.0 velocity=1.0 -> lower=-0.95 upper=2.1 effort=100.0 velocity=1.0
- joint joint3: limit lower=-1.50796447372 upper=3.0 effort=1000.0 velocity=1.0 -> lower=-1.50796447372 upper=3.0 effort=100.0 velocity=1.0
- joint joint4: limit lower=-1.57079632679 upper=1.57079632679 effort=1000.0 velocity=1.0 -> lower=-1.57079632679 upper=1.57079632679 effort=100.0 velocity=1.0

File: arips_ros/arips_arm_description/urdf/arips_arm.xacro (robot description, xacro)
@@ -133,5 +133,5 @@
     <axis xyz="0 1 0"/>
     <origin xyz="0 0 ${link3_len}"/>
-    <limit effort="1000.0" lower="${-pi*0.55}" upper="3.0" velocity="1.0"/>
+    <limit effort="1000.0" lower="-2.09" upper="2.09" velocity="1.0"/>
   </joint>
   <joint name="joint4" type="revolute">
@@ -140,5 +140,5 @@
     <axis xyz="0 1 0"/>
     <origin xyz="0 0 ${link4_len}"/>
-    <limit effort="1000.0" lower="${-pi/2}" upper="${pi/2}" velocity="1.0"/>
+    <limit effort="1000.0" lower="-2.09" upper="2.09" velocity="1.0"/>
   </joint>
   <joint name="joint5" type="revolute">
@@ -147,5 +147,5 @@
     <axis xyz="0 0 1"/>
     <origin xyz="0 0 ${link5_len / 2}"/>
-    <limit effort="1000.0" lower="${-pi/2}" upper="${pi/2}" velocity="1.0"/>
+    <limit effort="1000.0" lower="-3.1" upper="3.1" velocity="1.0"/>
   </joint>
   <joint name="link6-tool0" type="fixed">
@@ -164,5 +164,5 @@
     <axis xyz="0 0 1"/>
     <origin xyz="-0.055 0.02 0"/>
-    <limit effort="1000.0" lower="0.02" upper="${gripper_open_angle}" velocity="1.0"/>
+    <limit effort="1000.0" lower="-2.09" upper="2.09" velocity="1.0"/>
   </joint>
   <joint name="gripper_joint_right" type="revolute">
